File: hardware/laser-range-finder-v2-bricklet.kicad_pcb (KiCad board)
At the start: 2 copper layers, 48.2 x 35.6 mm, 30 parts, among them P1 CON-SENSOR2, P2 DEBUG, P3 BOOT, P4 JST_GHR_6, U1 XMC1XXX24, U2 DRILL, U3 DRILL, U4 DRILL, U5 DRILL

Commit message: changed processor to XMC1100
Parts:
- U1: value XMC1XXX24 -> XMC1100
Changed lines of the file:
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@@
   )
   (setup
-    (last_trace_width 0.5)
+    (last_trace_width 0.2)
     (user_trace_width 0.29972)
     (user_trace_width 0.3)
@@
       (effects (font (size 0.3 0.3) (thickness 0.075)))
     )
-    (fp_text value XMC1XXX24 (at 0 0.8 90) (layer F.Fab)
+    (fp_text value XMC1100 (at 0 0.8 90) (layer F.Fab)
       (effects (font (size 0.3 0.3) (thickness 0.075)))
     )
